Commit message: Add depth camera above gripper

File: ur5/ur5_description/urdf/ur5_robotiq85_gripper.urdf.xacro (robot description, xacro)
@@ -46,4 +46,54 @@
     <origin xyz="0 0 0.004" rpy="0 ${-pi/2} ${pi}"/>
   </xacro:robotiq_85_gripper>
+  <!-- Depth camera just above the gripper -->
+  <link name="depth_camera_link">
+    <visual>
+      <geometry>
+        <box size="0.02 0.02 0.02"/>
+      </geometry>
+      <material name="flat_black"/>
+    </visual>
+    <collision>
+      <geometry>
+        <box size="0.02 0.02 0.02"/>
+      </geometry>
+    </collision>
+    <inertial>
+      <origin xyz="0 0 0"/>
+      <mass value="0.01"/>
+      <inertia ixx="1e-6" ixy="0" ixz="0" iyy="1e-6" iyz="0" izz="1e-6"/>
+    </inertial>
+  </link>
+  <joint name="depth_camera_joint" type="fixed">
+    <origin xyz="0 0 0.10" rpy="0 0 0"/>
+    <parent link="robotiq_coupler"/>
+    <child link="depth_camera_link"/>
+  </joint>
+  <gazebo reference="depth_camera_link">
+    <sensor type="depth" name="depth_camera">
+      <update_rate>30.0</update_rate>
+      <camera name="depth_camera">
+        <horizontal_fov>1.047</horizontal_fov>
+        <image>
+          <width>640</width>
+          <height>480</height>
+          <format>R8G8B8</format>
+        </image>
+        <clip>
+          <near>0.05</near>
+          <far>5.0</far>
+        </clip>
+      </camera>
+      <plugin name="gazebo_depth_camera_controller" filename="libgazebo_ros_depth_camera.so">
+        <alwaysOn>true</alwaysOn>
+        <updateRate>30.0</updateRate>
+        <cameraName>depth_camera</cameraName>
+        <imageTopicName>image_raw</imageTopicName>
+        <cameraInfoTopicName>camera_info</cameraInfoTopicName>
+        <depthImageTopicName>depth/image_raw</depthImageTopicName>
+        <frameName>depth_camera_link</frameName>
+      </plugin>
+    </sensor>
+  </gazebo>
   <!-- Gazebo FT sensor plugin -->
   <gazebo reference="wrist_3_joint">

Commit message: Add depth camera above gripper

File: ur5/ur5_description/urdf/ur5_robotiq85_gripper.urdf.xacro (robot description, xacro)
@@ -71,3 +71,46 @@
     </gripper>
   </gazebo>
+  <!-- Depth camera mounted above the gripper -->
+  <link name="depth_camera_link">
+    <visual>
+      <geometry>
+        <box size="0.02 0.02 0.02"/>
+      </geometry>
+      <material name="flat_black"/>
+    </visual>
+    <inertial>
+      <origin xyz="0 0 0" rpy="0 0 0"/>
+      <mass value="0.1"/>
+      <inertia ixx="1e-5" ixy="0" ixz="0" iyy="1e-5" iyz="0" izz="1e-5"/>
+    </inertial>
+  </link>
+  <joint name="depth_camera_joint" type="fixed">
+    <parent link="robotiq_coupler"/>
+    <child link="depth_camera_link"/>
+    <origin xyz="0 0 0.10" rpy="0 0 0"/>
+  </joint>
+  <gazebo reference="depth_camera_link">
+    <sensor type="depth" name="depth_camera">
+      <update_rate>30.0</update_rate>
+      <camera>
+        <horizontal_fov>1.047</horizontal_fov>
+        <image>
+          <width>640</width>
+          <height>480</height>
+          <format>R8G8B8</format>
+        </image>
+        <clip>
+          <near>0.05</near>
+          <far>5.0</far>
+        </clip>
+      </camera>
+      <plugin name="depth_camera_controller" filename="libgazebo_ros_camera.so">
+        <cameraName>depth_camera</cameraName>
+        <frameName>depth_camera_link</frameName>
+        <imageTopicName>image_raw</imageTopicName>
+        <depthImageTopicName>depth/image_raw</depthImageTopicName>
+        <cameraInfoTopicName>camera_info</cameraInfoTopicName>
+      </plugin>
+    </sensor>
+  </gazebo>
 </robot>

Commit message: depth camera agregada

File: ur5/ur5_description/urdf/ur5_robotiq85_gripper.urdf.xacro (robot description, xacro)
@@ -88,5 +88,12 @@
     <parent link="robotiq_coupler"/>
     <child link="depth_camera_link"/>
-    <origin xyz="0 0 0.10" rpy="0 0 0"/>
+    <origin xyz="0.03 0 0.05" rpy="0 -1.5708 0"/>
+  </joint>
+  <link name="camera_link"/>
+  <joint name="camera_optical_joint" type="fixed">
+    <parent link="depth_camera_link"/>
+    <child  link="camera_link"/>
+    <!-- ROS optical frame: -90° sobre X, +90° sobre Z -->
+    <origin xyz="0 0 0" rpy="-1.5708 0 -1.5708"/>
   </joint>
   <gazebo reference="depth_camera_link">
@@ -105,11 +112,30 @@
         </clip>
       </camera>
-      <plugin name="depth_camera_controller" filename="libgazebo_ros_camera.so">
-        <cameraName>depth_camera</cameraName>
-        <frameName>depth_camera_link</frameName>
-        <imageTopicName>image_raw</imageTopicName>
-        <depthImageTopicName>depth/image_raw</depthImageTopicName>
-        <cameraInfoTopicName>camera_info</cameraInfoTopicName>
-      </plugin>
+        <plugin name="camera_plugin" filename="libgazebo_ros_openni_kinect.so">
+          <baseline>0.2</baseline>
+          <alwaysOn>true</alwaysOn>
+          <!-- Keep this zero, update_rate in the parent <sensor> tag
+            will control the frame rate. -->
+          <updateRate>0.0</updateRate>
+          <cameraName>camera_ir</cameraName>
+          <imageTopicName>/camera/color/image_raw</imageTopicName>
+          <cameraInfoTopicName>/camera/color/camera_info</cameraInfoTopicName>
+          <depthImageTopicName>/camera/depth/image_raw</depthImageTopicName>
+          <depthImageCameraInfoTopicName>/camera/depth/camera_info</depthImageCameraInfoTopicName>
+          <pointCloudTopicName>/camera/depth/points</pointCloudTopicName>
+          <frameName>camera_link</frameName>
+          <pointCloudCutoff>0.5</pointCloudCutoff>
+          <pointCloudCutoffMax>3.0</pointCloudCutoffMax>
+          <distortionK1>0</distortionK1>
+          <distortionK2>0</distortionK2>
+          <distortionK3>0</distortionK3>
+          <distortionT1>0</distortionT1>
+          <distortionT2>0</distortionT2>
+          <CxPrime>0</CxPrime>
+          <Cx>0</Cx>
+          <Cy>0</Cy>
+          <focalLength>0</focalLength>
+          <hackBaseline>0</hackBaseline>
+        </plugin>
     </sensor>
   </gazebo>

Commit message: scan shelves

File: ur5/ur5_description/urdf/ur5_robotiq85_gripper.urdf.xacro (robot description, xacro)
@@ -88,5 +88,5 @@
     <parent link="robotiq_coupler"/>
     <child link="depth_camera_link"/>
-    <origin xyz="0.03 0 0.05" rpy="0 -1.5708 0"/>
+    <origin xyz="-0.05 0 0.1" rpy="0 -1.5708 0"/>
   </joint>
   <link name="camera_link"/>
@@ -125,5 +125,5 @@
           <pointCloudTopicName>/camera/depth/points</pointCloudTopicName>
           <frameName>camera_link</frameName>
-          <pointCloudCutoff>0.15</pointCloudCutoff>
+          <pointCloudCutoff>0.05</pointCloudCutoff>
           <pointCloudCutoffMax>3.0</pointCloudCutoffMax>
           <distortionK1>0</distortionK1>
